Commit message: added cube at zero pos tip in 'SSRMS_Canadarm2.urdf', created 'objects.urdf'

File: urdf/SSRMS_Canadarm2.urdf (robot description, URDF)
Before this commit: robot SSRMS_Canadarm2, 10 links, 9 joints
Links:
- added link lcub, mass 1.0; collision box size=0.10 0.10 0.10
- added link lcub-xm; visual box size=0.0202 0.09 0.09
- added link lcub-xp; visual box size=0.0202 0.09 0.09
- added link lcub-ym; visual box size=0.09 0.0202 0.09
- added link lcub-yp; visual box size=0.09 0.0202 0.09
- added link lcub-zm; visual box size=0.09 0.09 0.0202
- added link lcub-zp; visual box size=0.09 0.09 0.0202
Joints:
- added joint attach-lcub: type fixed, parent world, child lcub, origin xyz=17.688 1.6134 0.0 rpy=-1.5708 0 1.5708
- added joint attach-lcub-xm: type fixed, parent lcub, child lcub-xm
- added joint attach-lcub-xp: type fixed, parent lcub, child lcub-xp
- added joint attach-lcub-ym: type fixed, parent lcub, child lcub-ym
- added joint attach-lcub-yp: type fixed, parent lcub, child lcub-yp
- added joint attach-lcub-zm: type fixed, parent lcub, child lcub-zm
- added joint attach-lcub-zp: type fixed, parent lcub, child lcub-zp

Commit message: ikin runs but needs weighted Jacobian, added green ball to tip of arm in urdf

File: urdf/SSRMS_Canadarm2.urdf (robot description, URDF)
Before this commit: robot SSRMS_Canadarm2, 17 links, 16 joints
Links:
- added link sphere; visual sphere radius=0.2
Joints:
- added joint attach-sphere: type fixed, parent link_ee, child sphere

Commit message: added paddle to Canadarm2 urdf

File: urdf/SSRMS_Canadarm2.urdf (robot description, URDF)
Before this commit: robot SSRMS_Canadarm2, 18 links, 17 joints
Links:
- removed link sphere
- added link paddle; visual cylinder length=0.1 radius=0.5
Joints:
- removed joint attach-sphere
- added joint attach-paddle: type fixed, parent link_ee, child paddle
